File: Main_Board.sch (EAGLE design)
At the start: 20 parts

Commit message: Added more parts
Parts:
- removed C2, C4: 100uF, SparkFun-Capacitors:CAP0805
- removed C5: (no value), SparkFun-Capacitors:CAP_POLG
- removed FRAME1: FRAME-LEDGER, SparkFun-Aesthetics:FRAME-LEDGER
- added FRAME2, FRAME3: FRAME-LETTER, SparkFun-Aesthetics:FRAME-LETTER
- added U$5: STM32F405RGT6, BB8:STM32F405RGT6
- added U$6, U$7: 100uF, BB8:CAP_POL_PAN
Connections:
- net GND: now also U$6.-, U$7.-; no longer C2.2, C4.2
- net VCC: now also U$6.+, U$7.+; no longer C2.1, C4.1
Other:
- note added: "Microcontroller"
- note added: "Motor Controllers"
Changed lines of the file:
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@@
 <part name="C1" library="SparkFun-Capacitors" deviceset="CAP" device="0805" value="470nF"/>
 <part name="GND4" library="SparkFun-Aesthetics" deviceset="GND" device=""/>
-<part name="C2" library="SparkFun-Capacitors" deviceset="CAP" device="0805" value="100uF"/>
 <part name="GND5" library="SparkFun-Aesthetics" deviceset="GND" device=""/>
 <part name="U$2" library="BB8" deviceset="BTM7752G" device=""/>
@@
 <part name="C3" library="SparkFun-Capacitors" deviceset="CAP" device="0805" value="470nF"/>
 <part name="GND9" library="SparkFun-Aesthetics" deviceset="GND" device=""/>
-<part name="C4" library="SparkFun-Capacitors" deviceset="CAP" device="0805" value="100uF"/>
 <part name="GND10" library="SparkFun-Aesthetics" deviceset="GND" device=""/>
-<part name="FRAME1" library="SparkFun-Aesthetics" deviceset="FRAME-LEDGER" device=""/>
-<part name="C5" library="SparkFun-Capacitors" deviceset="CAP_POL" device="G"/>
+<part name="U$5" library="BB8" deviceset="STM32F405RGT6" device=""/>
+<part name="FRAME2" library="SparkFun-Aesthetics" deviceset="FRAME-LETTER" device=""/>
+<part name="FRAME3" library="SparkFun-Aesthetics" deviceset="FRAME-LETTER" device=""/>
+<part name="U$6" library="BB8" deviceset="CAP_POL_PAN" device="" value="100uF"/>
+<part name="U$7" library="BB8" deviceset="CAP_POL_PAN" device="" value="100uF"/>
 </parts>
 <sheets>
 <sheet>
 <plain>
+<text x="83.82" y="170.18" size="6.4516" layer="95">Motor Controllers </text>
+<text x="365.76" y="170.18" size="6.4516" layer="95">Microcontroller</text>
 </plain>
 <instances>
@@
 <instance part="C1" gate="G$1" x="17.78" y="114.3"/>
 <instance part="GND4" gate="1" x="17.78" y="106.68"/>
-<instance part="C2" gate="G$1" x="7.62" y="114.3"/>
 <instance part="GND5" gate="1" x="7.62" y="106.68"/>
 <instance part="U$2" gate="G$1" x="58.42" y="27.94"/>
@@
 <instance part="C3" gate="G$1" x="17.78" y="43.18"/>
 <instance part="GND9" gate="1" x="17.78" y="35.56"/>
-<instance part="C4" gate="G$1" x="7.62" y="43.18"/>
 <instance part="GND10" gate="1" x="7.62" y="35.56"/>
-<instance part="FRAME1" gate="G$1" x="-10.16" y="-12.7"/>
-<instance part="FRAME1" gate="G$2" x="320.04" y="-12.7"/>
-<instance part="C5" gate="G$1" x="2.54" y="58.42"/>
+<instance part="U$5" gate="G$1" x="386.08" y="104.14"/>
+<instance part="FRAME2" gate="G$1" x="-7.62" y="-5.08"/>
+<instance part="FRAME2" gate="V" x="139.7" y="-5.08"/>
+<instance part="FRAME3" gate="G$1" x="264.16" y="-5.08"/>
+<instance part="FRAME3" gate="V" x="411.48" y="-5.08"/>
+<instance part="U$6" gate="G$1" x="7.62" y="116.84"/>
+<instance part="U$7" gate="G$1" x="7.62" y="45.72"/>
 </instances>
 <busses>
@@
 <wire x1="17.78" y1="119.38" x2="17.78" y2="121.92" width="0.1524" layer="91"/>
 <wire x1="17.78" y1="121.92" x2="30.48" y2="121.92" width="0.1524" layer="91"/>
-<pinref part="C2" gate="G$1" pin="1"/>
-<wire x1="7.62" y1="119.38" x2="7.62" y2="121.92" width="0.1524" layer="91"/>
 <wire x1="7.62" y1="121.92" x2="17.78" y2="121.92" width="0.1524" layer="91"/>
 <junction x="17.78" y="121.92"/>
+<pinref part="U$6" gate="G$1" pin="+"/>
+<wire x1="7.62" y1="121.92" x2="7.62" y2="119.38" width="0.1524" layer="91"/>
 </segment>
 <segment>
@@
 <wire x1="17.78" y1="48.26" x2="17.78" y2="50.8" width="0.1524" layer="91"/>
 <wire x1="17.78" y1="50.8" x2="30.48" y2="50.8" width="0.1524" layer="91"/>
-<pinref part="C4" gate="G$1" pin="1"/>
-<wire x1="7.62" y1="48.26" x2="7.62" y2="50.8" width="0.1524" layer="91"/>
 <wire x1="7.62" y1="50.8" x2="17.78" y2="50.8" width="0.1524" layer="91"/>
 <junction x="17.78" y="50.8"/>
+<pinref part="U$7" gate="G$1" pin="+"/>
+<wire x1="7.62" y1="50.8" x2="7.62" y2="48.26" width="0.1524" layer="91"/>
 </segment>
 </net>
@@
 </segment>
 <segment>
-<pinref part="GND5" gate="1" pin="GND"/>
-<pinref part="C2" gate="G$1" pin="2"/>
-<wire x1="7.62" y1="109.22" x2="7.62" y2="111.76" width="0.1524" layer="91"/>
-</segment>
-<segment>
 <pinref part="U$2" gate="G$1" pin="GND@25"/>
 <pinref part="GND6" gate="1" pin="GND"/>
@@
 </segment>
 <segment>
+<pinref part="U$6" gate="G$1" pin="-"/>
+<pinref part="GND5" gate="1" pin="GND"/>
+<wire x1="7.62" y1="111.76" x2="7.62" y2="109.22" width="0.1524" layer="91"/>
+</segment>
+<segment>
+<pinref part="U$7" gate="G$1" pin="-"/>
 <pinref part="GND10" gate="1" pin="GND"/>
-<pinref part="C4" gate="G$1" pin="2"/>
-<wire x1="7.62" y1="38.1" x2="7.62" y2="40.64" width="0.1524" layer="91"/>
+<wire x1="7.62" y1="40.64" x2="7.62" y2="38.1" width="0.1524" layer="91"/>
 </segment>
 </net>

Commit message: Updated board
Parts:
- added U1: RN4020RN4020, BB8:RN4020RN4020
Changed lines of the file:
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@@
 <part name="U$6" library="BB8" deviceset="CAP_POL_PAN" device="" value="100uF"/>
 <part name="U$7" library="BB8" deviceset="CAP_POL_PAN" device="" value="100uF"/>
+<part name="U1" library="BB8" deviceset="RN4020" device="RN4020"/>
 </parts>
 <sheets>
@@
 <instance part="U$6" gate="G$1" x="7.62" y="116.84"/>
 <instance part="U$7" gate="G$1" x="7.62" y="45.72"/>
+<instance part="U1" gate="G$1" x="22.86" y="-76.2"/>
 </instances>
 <busses>

Commit message: Started powering micro
Parts:
- removed FRAME3: FRAME-LETTER, SparkFun-Aesthetics:FRAME-LETTER
- added C10: 1uF, SparkFun-Capacitors:CAP0805
- added C11, C12: 2.2uF, SparkFun-Capacitors:CAP0805
- added C2: 10uF, SparkFun-Capacitors:CAP0805
- added C4, C5, C6, C7, C8, C9: 100nF, SparkFun-Capacitors:CAP0805
- added FRAME4: FRAME-LEDGER, SparkFun-Aesthetics:FRAME-LEDGER
- FRAME2: value FRAME-LETTER -> FRAME-LEDGER; device SparkFun-Aesthetics:FRAME-LETTER -> SparkFun-Aesthetics:FRAME-LEDGER
Connections:
- new net 3.3V: C10.2, C2.1, C4.1, C5.1, C6.1, C7.1, C8.1, C9.2, U$5.VBAT, U$5.VDD, U$5.VDD@32, U$5.VDD@48, U$5.VDD@64, U$5.VDDA
- new net N$15: C12.1, U$5.VCAP_2
- new net N$16: C11.1, U$5.VCAP_1
- net GND: now also C10.1, C11.2, C12.2, C2.2, C4.2, C5.2, C6.2, C7.2, C8.2, C9.1, U$5.VSS, U$5.VSS@63, U$5.VSSA
Other:
- moved on the sheet: U$5

Commit message: Labeling MCs
Parts:
- added C13, C14: (no value), SparkFun-Capacitors:CAP0805
- added FRAME1, FRAME3: FRAME-LEDGER, SparkFun-Aesthetics:FRAME-LEDGER
- added U$8: LMS8117, BB8:LMS8117
Connections:
- net N$12 renamed MC2_IS
- net N$7 renamed MC1_IS
- new net MC1_IN1: R1.1
- new net MC1_IN2: R2.1
- new net MC1_INH: R3.2
- new net MC2_IN1: R6.1
- new net MC2_IN2: R7.1
- new net MC2_INH: R8.2
- net 3.3V: now also C14.1, U$8.VOUT
- net 5V: now also C13.1, U$8.VIN
- net GND: now also C13.2, C14.2, U$8.ADJ/GND
Other:
- note added: "Bluetooth"
- note added: "Power Conversion"
- moved on the sheet: U1
Changed lines of the file:
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@@
 <part name="FRAME2" library="SparkFun-Aesthetics" deviceset="FRAME-LEDGER" device=""/>
 <part name="FRAME4" library="SparkFun-Aesthetics" deviceset="FRAME-LEDGER" device=""/>
+<part name="FRAME1" library="SparkFun-Aesthetics" deviceset="FRAME-LEDGER" device=""/>
+<part name="FRAME3" library="SparkFun-Aesthetics" deviceset="FRAME-LEDGER" device=""/>
+<part name="U$8" library="BB8" deviceset="LMS8117" device=""/>
+<part name="SUPPLY12" library="SparkFun-Aesthetics" deviceset="5V" device=""/>
+<part name="GND17" library="SparkFun-Aesthetics" deviceset="GND" device=""/>
+<part name="SUPPLY13" library="SparkFun-Aesthetics" deviceset="3.3V" device=""/>
+<part name="C13" library="SparkFun-Capacitors" deviceset="CAP" device="0805"/>
+<part name="C14" library="SparkFun-Capacitors" deviceset="CAP" device="0805"/>
+<part name="GND18" library="SparkFun-Aesthetics" deviceset="GND" device=""/>
 </parts>
 <sheets>
@@
 <text x="0" y="223.52" size="6.4516" layer="95">Motor Controllers </text>
 <text x="495.3" y="223.52" size="6.4516" layer="95">Microcontroller</text>
+<text x="7.62" y="-66.04" size="6.4516" layer="95">Power Conversion</text>
+<text x="472.44" y="-71.12" size="6.4516" layer="95">Bluetooth</text>
 </plain>
 <instances>
@@
 <instance part="U$6" gate="G$1" x="7.62" y="116.84"/>
 <instance part="U$7" gate="G$1" x="7.62" y="45.72"/>
-<instance part="U1" gate="G$1" x="22.86" y="-76.2"/>
+<instance part="U1" gate="G$1" x="495.3" y="-266.7"/>
 <instance part="SUPPLY5" gate="G$1" x="287.02" y="50.8"/>
 <instance part="SUPPLY6" gate="G$1" x="312.42" y="5.08"/>
@@
 <instance part="FRAME4" gate="G$1" x="-172.72" y="-43.18"/>
 <instance part="FRAME4" gate="G$2" x="157.48" y="-43.18"/>
+<instance part="FRAME1" gate="G$1" x="-170.18" y="-335.28"/>
+<instance part="FRAME1" gate="G$2" x="157.48" y="-332.74"/>
+<instance part="FRAME3" gate="G$1" x="274.32" y="-335.28"/>
+<instance part="FRAME3" gate="G$2" x="601.98" y="-335.28"/>
+<instance part="U$8" gate="G$1" x="-104.14" y="-93.98"/>
+<instance part="SUPPLY12" gate="G$1" x="-129.54" y="-88.9"/>
+<instance part="GND17" gate="1" x="-129.54" y="-106.68"/>
+<instance part="SUPPLY13" gate="G$1" x="-71.12" y="-91.44"/>
+<instance part="C13" gate="G$1" x="-124.46" y="-99.06"/>
+<instance part="C14" gate="G$1" x="-71.12" y="-99.06"/>
+<instance part="GND18" gate="1" x="-71.12" y="-106.68"/>
 </instances>
 <busses>
@@
 <wire x1="396.24" y1="12.7" x2="403.86" y2="12.7" width="0.1524" layer="91"/>
 </segment>
+<segment>
+<pinref part="C13" gate="G$1" pin="2"/>
+<pinref part="U$8" gate="G$1" pin="ADJ/GND"/>
+<wire x1="-124.46" y1="-101.6" x2="-109.22" y2="-101.6" width="0.1524" layer="91"/>
+<pinref part="GND17" gate="1" pin="GND"/>
+<wire x1="-129.54" y1="-104.14" x2="-129.54" y2="-101.6" width="0.1524" layer="91"/>
+<wire x1="-129.54" y1="-101.6" x2="-124.46" y2="-101.6" width="0.1524" layer="91"/>
+<junction x="-124.46" y="-101.6"/>
+</segment>
+<segment>
+<pinref part="C14" gate="G$1" pin="2"/>
+<pinref part="GND18" gate="1" pin="GND"/>
+<wire x1="-71.12" y1="-101.6" x2="-71.12" y2="-104.14" width="0.1524" layer="91"/>
+</segment>
 </net>
 <net name="N$1" class="0">
@@
 </segment>
 </net>
-<net name="N$7" class="0">
+<net name="MC1_IS" class="0">
 <segment>
 <pinref part="R4" gate="G$1" pin="2"/>
@@
 <junction x="111.76" y="78.74"/>
 <wire x1="111.76" y1="88.9" x2="121.92" y2="88.9" width="0.1524" layer="91"/>
+<label x="116.84" y="88.9" size="1.778" layer="95"/>
 </segment>
 </net>
@@
 <wire x1="104.14" y1="50.8" x2="101.6" y2="50.8" width="0.1524" layer="91"/>
 <wire x1="101.6" y1="50.8" x2="101.6" y2="58.42" width="0.1524" layer="91"/>
+</segment>
+<segment>
+<pinref part="U$8" gate="G$1" pin="VIN"/>
+<pinref part="C13" gate="G$1" pin="1"/>
+<wire x1="-109.22" y1="-93.98" x2="-124.46" y2="-93.98" width="0.1524" layer="91"/>
+<pinref part="SUPPLY12" gate="G$1" pin="5V"/>
+<wire x1="-124.46" y1="-93.98" x2="-129.54" y2="-93.98" width="0.1524" layer="91"/>
+<wire x1="-129.54" y1="-93.98" x2="-129.54" y2="-88.9" width="0.1524" layer="91"/>
+<junction x="-124.46" y="-93.98"/>
 </segment>
 </net>
@@
 </segment>
 </net>
-<net name="N$12" class="0">
+<net name="MC2_IS" class="0">
 <segment>
 <pinref part="R9" gate="G$1" pin="2"/>
@@
 <junction x="111.76" y="7.62"/>
 <wire x1="111.76" y1="17.78" x2="121.92" y2="17.78" width="0.1524" layer="91"/>
+<label x="114.3" y="17.78" size="1.778" layer="95"/>
 </segment>
 </net>
@@
 <junction x="525.78" y="134.62"/>
 </segment>
+<segment>
+<pinref part="U$8" gate="G$1" pin="VOUT"/>
+<pinref part="C14" gate="G$1" pin="1"/>
+<wire x1="-81.28" y1="-93.98" x2="-71.12" y2="-93.98" width="0.1524" layer="91"/>
+<pinref part="SUPPLY13" gate="G$1" pin="3.3V"/>
+<wire x1="-71.12" y1="-93.98" x2="-71.12" y2="-91.44" width="0.1524" layer="91"/>
+<junction x="-71.12" y="-93.98"/>
+</segment>
 </net>
 <net name="N$15" class="0">
@@
 </segment>
 </net>
+<net name="MC2_IN1" class="0">
+<segment>
+<pinref part="R6" gate="G$1" pin="1"/>
+<wire x1="-2.54" y1="30.48" x2="-10.16" y2="30.48" width="0.1524" layer="91"/>
+<label x="-15.24" y="30.48" size="1.778" layer="95"/>
+</segment>
+</net>
+<net name="MC2_IN2" class="0">
+<segment>
+<pinref part="R7" gate="G$1" pin="1"/>
+<wire x1="7.62" y1="27.94" x2="-10.16" y2="27.94" width="0.1524" layer="91"/>
+<label x="-15.24" y="27.94" size="1.778" layer="95"/>
+</segment>
+</net>
+<net name="MC1_IN1" class="0">
+<segment>
+<pinref part="R1" gate="G$1" pin="1"/>
+<wire x1="-2.54" y1="101.6" x2="-10.16" y2="101.6" width="0.1524" layer="91"/>
+<label x="-12.7" y="101.6" size="1.778" layer="95"/>
+</segment>
+</net>
+<net name="MC1_IN2" class="0">
+<segment>
+<pinref part="R2" gate="G$1" pin="1"/>
+<wire x1="7.62" y1="99.06" x2="-10.16" y2="99.06" width="0.1524" layer="91"/>
+<label x="-12.7" y="99.06" size="1.778" layer="95"/>
+</segment>
+</net>
+<net name="MC1_INH" class="0">
+<segment>
+<pinref part="R3" gate="G$1" pin="2"/>
+<wire x1="96.52" y1="81.28" x2="96.52" y2="83.82" width="0.1524" layer="91"/>
+<wire x1="96.52" y1="83.82" x2="106.68" y2="83.82" width="0.1524" layer="91"/>
+<label x="99.06" y="83.82" size="1.778" layer="95"/>
+</segment>
+</net>
+<net name="MC2_INH" class="0">
+<segment>
+<pinref part="R8" gate="G$1" pin="2"/>
+<wire x1="96.52" y1="10.16" x2="96.52" y2="12.7" width="0.1524" layer="91"/>
+<wire x1="96.52" y1="12.7" x2="106.68" y2="12.7" width="0.1524" layer="91"/>
+<label x="99.06" y="12.7" size="1.778" layer="95"/>
+</segment>
+</net>

Commit message: Added leve; translation for motor stuff
Parts:
- added U$10, U$9: SN74LV4T125, BB8:SN74LV4T125
Connections:
- removed net MC1_INH: R3.2
- removed net MC2_INH: R8.2
- new net M1_A_3.3: U$9.1Y
- new net M1_A_5: U$3.A, U$9.1A
- new net M1_B_3.3: U$9.2Y
- new net M1_B_5: U$3.B, U$9.2A
- new net M2_A_3.3: U$9.4Y
- new net M2_A_5: U$4.A, U$9.4A
- new net M2_B_3.3: U$9.3Y
- new net M2_B_5: U$4.B, U$9.3A
- new net MC1_ING_3.3: U$10.2A
- new net MC1_INH_3.3: U$10.1A
- new net MC1_INH_5: R3.2, U$10.1Y
- new net MC2_INH_5: R8.2, U$10.2Y
- net 3.3V: now also U$9.VCC
- net 5V: now also U$10.3!OE, U$10.4!OE, U$10.VCC
- net GND: now also U$10.1!OE, U$10.2!OE, U$10.3A, U$10.4A, U$10.GND, U$9.1!OE, U$9.2!OE, U$9.3!OE, U$9.4!OE, U$9.GND
Other:
- note added: "Micro Input from MC: M1_A_3.3 M1_B_3.3 M2_A_3.3 M2_B_3.3 MC1_IS MC2_IS Micro Output to MC MC1_INH_3.3 MC2_INH_3.3"

Commit message: Updates
Parts:
- added C15: 4.7uF, SparkFun-Capacitors:CAP0805
Connections:
- net 3.3V: now also C15.2, U1.VDD
- net GND: now also C15.1, U1.GND@1, U1.GND@24
Other:
- moved on the sheet: U1
Changed lines of the file:
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@@
 <part name="SUPPLY16" library="SparkFun-Aesthetics" deviceset="5V" device=""/>
 <part name="SUPPLY17" library="SparkFun-Aesthetics" deviceset="5V" device=""/>
+<part name="SUPPLY18" library="SparkFun-Aesthetics" deviceset="3.3V" device=""/>
+<part name="C15" library="SparkFun-Capacitors" deviceset="CAP" device="0805" value="4.7uF"/>
+<part name="GND29" library="SparkFun-Aesthetics" deviceset="GND" device=""/>
+<part name="GND30" library="SparkFun-Aesthetics" deviceset="GND" device=""/>
+<part name="GND31" library="SparkFun-Aesthetics" deviceset="GND" device=""/>
 </parts>
 <sheets>
@@
 <instance part="U$6" gate="G$1" x="7.62" y="116.84"/>
 <instance part="U$7" gate="G$1" x="7.62" y="45.72"/>
-<instance part="U1" gate="G$1" x="495.3" y="-266.7"/>
+<instance part="U1" gate="G$1" x="505.46" y="-175.26"/>
 <instance part="SUPPLY5" gate="G$1" x="287.02" y="50.8"/>
 <instance part="SUPPLY6" gate="G$1" x="312.42" y="5.08"/>
@@
 <instance part="SUPPLY16" gate="G$1" x="193.04" y="50.8"/>
 <instance part="SUPPLY17" gate="G$1" x="193.04" y="35.56"/>
+<instance part="SUPPLY18" gate="G$1" x="546.1" y="-147.32"/>
+<instance part="C15" gate="G$1" x="566.42" y="-154.94" rot="R180"/>
+<instance part="GND29" gate="1" x="467.36" y="-157.48"/>
+<instance part="GND30" gate="1" x="538.48" y="-157.48"/>
+<instance part="GND31" gate="1" x="566.42" y="-165.1"/>
 </instances>
 <busses>
@@
 <wire x1="193.04" y1="30.48" x2="185.42" y2="30.48" width="0.1524" layer="91"/>
 </segment>
+<segment>
+<pinref part="U1" gate="G$1" pin="GND@24"/>
+<pinref part="GND30" gate="1" pin="GND"/>
+<wire x1="533.4" y1="-154.94" x2="538.48" y2="-154.94" width="0.1524" layer="91"/>
+</segment>
+<segment>
+<pinref part="C15" gate="G$1" pin="1"/>
+<pinref part="GND31" gate="1" pin="GND"/>
+<wire x1="566.42" y1="-162.56" x2="566.42" y2="-160.02" width="0.1524" layer="91"/>
+</segment>
+<segment>
+<pinref part="U1" gate="G$1" pin="GND@1"/>
+<pinref part="GND29" gate="1" pin="GND"/>
+<wire x1="477.52" y1="-154.94" x2="467.36" y2="-154.94" width="0.1524" layer="91"/>
+</segment>
 </net>
 <net name="N$1" class="0">
@@
 <wire x1="193.04" y1="129.54" x2="193.04" y2="132.08" width="0.1524" layer="91"/>
 </segment>
-</net>
+<segment>
+<pinref part="U1" gate="G$1" pin="VDD"/>
+<wire x1="533.4" y1="-160.02" x2="546.1" y2="-160.02" width="0.1524" layer="91"/>
+<pinref part="SUPPLY18" gate="G$1" pin="3.3V"/>
+<wire x1="546.1" y1="-160.02" x2="546.1" y2="-149.86" width="0.1524" layer="91"/>
+<pinref part="C15" gate="G$1" pin="2"/>
+<wire x1="546.1" y1="-149.86" x2="546.1" y2="-147.32" width="0.1524" layer="91"/>
+<wire x1="566.42" y1="-152.4" x2="566.42" y2="-149.86" width="0.1524" layer="91"/>
+<wire x1="566.42" y1="-149.86" x2="546.1" y2="-149.86" width="0.1524" layer="91"/>
+<junction x="546.1" y="-149.86"/>
+</segment>
+</net>
