File: Main_Board.sch (EAGLE design)
At the start: 216 parts, among them J1 SERVO, J2 5.5x2.1mm Barrel, J3 9.7uH, J4 BATTERY, J5 SPEAKER, J6 SD_WP, P1 MOTOR_HEADER, P2 MOTOR_HEADER, P3 JTAG, P4 5738-SDCARD, Q1 SI9933CDY-PFET, Q2 CSD17308Q3, Q3 CSD17308Q3, Q4 CSD17308Q3, Q5 CSD17308Q3, Q6 CSD17308Q3, Q7 CSD17308Q3, Q8 CSD17308Q3, U1 LMS8117, U10 IMU, U11 LTC3122-MSOP, U12 CBAT54S-SOT23-3, U13 BQ2947, U14 TPA2005D1DGN, U15 BQ40Z60, U2 5V_BUCK_REG, U3 BTM7752G, U4 BTM7752G, U5 SN74LV4T125, U6 SN74LV4T125, U7 STM32F405RGT6, U8 RN4020RN4020, U9 BQ51013B-20VQFN

Commit message: replaced SPI sd to SDIO
Parts:
- removed P4: 5738-SDCARD, BB8:5738-SDCARD
- J6: value SD_WP -> SDIO-SDCARD; device SparkFun-Connectors:M02PTH -> BB8:SDIO-SDCARD
Connections:
- removed net N$41: J6.1, P4.WP
- removed net N$42: J6.2, P4.COM
- removed net SD_SPI_MISO: P4.MISO, U7.PC2
- removed net SD_SPI_MOSI: P4.MOSI, U7.PC3
- removed net SD_SPI_NSS: P4.CS, U7.PB9
- removed net SD_SPI_SCK: P4.CLK, U7.PB13
- new net SDIO_CK: J6.CLK, U7.PC12
- new net SDIO_CMD: J6.CMD, U7.PD2
- new net SDIO_D0: J6.DATA, U7.PC8
- net GND: now also J6.GND@3, J6.GND@6; no longer P4.GND@3, P4.GND@6
- net MC2_INH_3.3: now also U7.PA12; no longer U7.PC8
- net N$27: now also J6.VCC; no longer P4.VCC
Changed lines of the file:
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@@
 <part name="GND65" library="SparkFun-Aesthetics" deviceset="GND" device=""/>
 <part name="U14" library="SparkFun-AnalogIC" deviceset="TPA2005D1" device="DGN"/>
-<part name="P4" library="BB8" deviceset="5738-SDCARD" device=""/>
 <part name="SUPPLY25" library="SparkFun-Aesthetics" deviceset="VCC" device=""/>
 <part name="GND72" library="SparkFun-Aesthetics" deviceset="GND" device=""/>
@@
 <part name="D1" library="SparkFun-LED" deviceset="LED-BLUE" device="0603" value="GREEN"/>
 <part name="GND28" library="SparkFun-Aesthetics" deviceset="GND" device=""/>
-<part name="J6" library="SparkFun-Connectors" deviceset="M02" device="PTH" value="SD_WP"/>
 <part name="SUPPLY26" library="SparkFun-Aesthetics" deviceset="VCC" device=""/>
+<part name="J6" library="BB8" deviceset="SDIO-SDCARD" device=""/>
 </parts>
 <sheets>
@@
 <instance part="GND65" gate="1" x="1503.68" y="114.3"/>
 <instance part="U14" gate="G$1" x="1455.42" y="111.76"/>
-<instance part="P4" gate="G$1" x="1605.28" y="111.76"/>
 <instance part="SUPPLY25" gate="G$1" x="1579.88" y="137.16"/>
 <instance part="GND72" gate="1" x="1584.96" y="81.28"/>
@@
 <instance part="D1" gate="G$1" x="314.96" y="134.62" rot="R270"/>
 <instance part="GND28" gate="1" x="289.56" y="132.08"/>
-<instance part="J6" gate="G$1" x="1645.92" y="124.46" rot="R180"/>
 <instance part="SUPPLY26" gate="G$1" x="1678.94" y="-88.9"/>
+<instance part="J6" gate="G$1" x="1605.28" y="111.76"/>
 </instances>
 <busses>
@@
 </segment>
 <segment>
-<pinref part="P4" gate="G$1" pin="GND@3"/>
 <pinref part="GND72" gate="1" pin="GND"/>
 <wire x1="1592.58" y1="91.44" x2="1584.96" y2="91.44" width="0.1524" layer="91"/>
 <wire x1="1584.96" y1="91.44" x2="1584.96" y2="86.36" width="0.1524" layer="91"/>
-<pinref part="P4" gate="G$1" pin="GND@6"/>
 <wire x1="1584.96" y1="86.36" x2="1584.96" y2="83.82" width="0.1524" layer="91"/>
 <wire x1="1592.58" y1="86.36" x2="1584.96" y2="86.36" width="0.1524" layer="91"/>
 <junction x="1584.96" y="86.36"/>
+<pinref part="J6" gate="G$1" pin="GND@3"/>
+<pinref part="J6" gate="G$1" pin="GND@6"/>
 </segment>
 <segment>
@@
 <net name="N$27" class="0">
 <segment>
-<pinref part="P4" gate="G$1" pin="VCC"/>
 <wire x1="1592.58" y1="132.08" x2="1579.88" y2="132.08" width="0.1524" layer="91"/>
 <wire x1="1579.88" y1="132.08" x2="1579.88" y2="137.16" width="0.1524" layer="91"/>
 <pinref part="SUPPLY25" gate="G$1" pin="VCC"/>
+<pinref part="J6" gate="G$1" pin="VCC"/>
 </segment>
 </net>
@@
 <net name="MC2_INH_3.3" class="0">
 <segment>
-<pinref part="U7" gate="G$1" pin="PC8"/>
-<wire x1="383.54" y1="73.66" x2="406.4" y2="73.66" width="0.1524" layer="91"/>
-<label x="396.24" y="73.66" size="1.778" layer="95"/>
-</segment>
-<segment>
 <pinref part="U6" gate="G$1" pin="2A"/>
 <wire x1="152.4" y1="35.56" x2="137.16" y2="35.56" width="0.1524" layer="91"/>
 <label x="137.16" y="35.56" size="1.778" layer="95"/>
 </segment>
+<segment>
+<pinref part="U7" gate="G$1" pin="PA12"/>
+<wire x1="383.54" y1="119.38" x2="411.48" y2="119.38" width="0.1524" layer="91"/>
+<label x="396.24" y="119.38" size="1.778" layer="95"/>
+</segment>
 </net>
 <net name="AC2" class="0">
@@
 </segment>
 </net>
-<net name="N$41" class="0">
-<segment>
-<pinref part="P4" gate="G$1" pin="WP"/>
-<wire x1="1620.52" y1="127" x2="1638.3" y2="127" width="0.1524" layer="91"/>
-<pinref part="J6" gate="G$1" pin="1"/>
-<wire x1="1638.3" y1="127" x2="1638.3" y2="124.46" width="0.1524" layer="91"/>
-</segment>
-</net>
-<net name="N$42" class="0">
-<segment>
-<pinref part="P4" gate="G$1" pin="COM"/>
-<wire x1="1620.52" y1="121.92" x2="1638.3" y2="121.92" width="0.1524" layer="91"/>
-<pinref part="J6" gate="G$1" pin="2"/>
-</segment>
-</net>
 <net name="AUDIO_PWM" class="0">
 <segment>
@@
 </segment>
 </net>
-<net name="SD_SPI_NSS" class="0">
-<segment>
-<pinref part="P4" gate="G$1" pin="CS"/>
-<wire x1="1592.58" y1="127" x2="1579.88" y2="127" width="0.1524" layer="91"/>
-<label x="1579.88" y="127" size="1.778" layer="95"/>
-</segment>
-<segment>
-<pinref part="U7" gate="G$1" pin="PB9"/>
-<wire x1="335.28" y1="165.1" x2="317.5" y2="165.1" width="0.1524" layer="91"/>
-<label x="317.5" y="165.1" size="1.778" layer="95"/>
-</segment>
-</net>
-<net name="SD_SPI_SCK" class="0">
-<segment>
-<pinref part="P4" gate="G$1" pin="CLK"/>
-<wire x1="1592.58" y1="121.92" x2="1579.88" y2="121.92" width="0.1524" layer="91"/>
-<label x="1579.88" y="121.92" size="1.778" layer="95"/>
-</segment>
-<segment>
-<pinref part="U7" gate="G$1" pin="PB13"/>
-<wire x1="383.54" y1="35.56" x2="406.4" y2="35.56" width="0.1524" layer="91"/>
-<label x="396.24" y="35.56" size="1.778" layer="95"/>
-</segment>
-</net>
-<net name="SD_SPI_MOSI" class="0">
-<segment>
-<pinref part="P4" gate="G$1" pin="MOSI"/>
-<wire x1="1592.58" y1="111.76" x2="1579.88" y2="111.76" width="0.1524" layer="91"/>
-<label x="1579.88" y="111.76" size="1.778" layer="95"/>
-</segment>
-<segment>
-<pinref part="U7" gate="G$1" pin="PC3"/>
-<wire x1="335.28" y1="66.04" x2="312.42" y2="66.04" width="0.1524" layer="91"/>
-<label x="314.96" y="66.04" size="1.778" layer="95"/>
-</segment>
-</net>
-<net name="SD_SPI_MISO" class="0">
-<segment>
-<pinref part="P4" gate="G$1" pin="MISO"/>
-<wire x1="1592.58" y1="106.68" x2="1579.88" y2="106.68" width="0.1524" layer="91"/>
-<label x="1579.88" y="106.68" size="1.778" layer="95"/>
-</segment>
-<segment>
-<pinref part="U7" gate="G$1" pin="PC2"/>
-<wire x1="335.28" y1="73.66" x2="312.42" y2="73.66" width="0.1524" layer="91"/>
-<label x="314.96" y="73.66" size="1.778" layer="95"/>
-</segment>
-</net>
 <net name="IMU_I2C_SDA" class="0">
 <segment>
@@
 </segment>
 </net>
+<net name="SDIO_D0" class="0">
+<segment>
+<pinref part="U7" gate="G$1" pin="PC8"/>
+<wire x1="383.54" y1="73.66" x2="406.4" y2="73.66" width="0.1524" layer="91"/>
+<label x="396.24" y="73.66" size="1.778" layer="95"/>
+</segment>
+<segment>
+<pinref part="J6" gate="G$1" pin="DATA"/>
+<wire x1="1592.58" y1="116.84" x2="1569.72" y2="116.84" width="0.1524" layer="91"/>
+<label x="1569.72" y="116.84" size="1.778" layer="95"/>
+</segment>
+</net>
+<net name="SDIO_CK" class="0">
+<segment>
+<pinref part="U7" gate="G$1" pin="PC12"/>
+<wire x1="383.54" y1="172.72" x2="414.02" y2="172.72" width="0.1524" layer="91"/>
+<label x="403.86" y="172.72" size="1.778" layer="95"/>
+</segment>
+<segment>
+<pinref part="J6" gate="G$1" pin="CLK"/>
+<wire x1="1592.58" y1="121.92" x2="1569.72" y2="121.92" width="0.1524" layer="91"/>
+<label x="1569.72" y="121.92" size="1.778" layer="95"/>
+</segment>
+</net>
+<net name="SDIO_CMD" class="0">
+<segment>
+<pinref part="U7" gate="G$1" pin="PD2"/>
+<wire x1="383.54" y1="165.1" x2="414.02" y2="165.1" width="0.1524" layer="91"/>
+<label x="403.86" y="165.1" size="1.778" layer="95"/>
+</segment>
+<segment>
+<pinref part="J6" gate="G$1" pin="CMD"/>
+<wire x1="1592.58" y1="127" x2="1569.72" y2="127" width="0.1524" layer="91"/>
+<label x="1569.72" y="127" size="1.778" layer="95"/>
+</segment>
+</net>
