File: ChargingCircuit.sch (EAGLE design)
At the start: 22 parts, among them U1 MAX745EACSSOP

Commit message: minor changes to charging board
Parts:
- removed U$1: IRF7303, Work:IRF7303
- removed U$2, U$3: MBRS340T3, Work:MBRS340T3
- removed U$4: THM, Work:THM
- added D2, D3: MBRS340T3, BB8:MBRS340T3
- added M1: IRF7303, BB8:IRF7303
- added THM1: (no value), BB8:THM
- C1: value (none) -> 68uF
- C2, C4, C6, C7: value (none) -> 0.1uF
- C3: value (none) -> 47nF
- D1: value 1N4148 -> 1N4148-0805; device SparkFun-DiscreteSemi:DIODE1N4148 -> BB8:1N4148-0805
- R11, R3: value (none) -> 100k
- R15, R2: value (none) -> 10k
Connections:
- net GND: now also D2.A, M1B.S, THM1.1; no longer U$1G$2.S, U$2.A, U$4.1
- net N$14: now also THM1.2; no longer U$4.2
- net N$3: now also M1A.G; no longer U$1G$1.G
- net N$4: now also M1B.G; no longer U$1G$2.G
- net N$5: now also D3.C; no longer U$3.C
- net N$6: now also D3.A; no longer U$3.A
- net N$8: now also D2.C, M1A.S, M1B.D; no longer U$1G$1.S, U$1G$2.D, U$2.C
- net VIN: now also M1A.D; no longer U$1G$1.D
Other:
- moved on the sheet: C1, C3, L1, R1, R15

Commit message: Added wireless charging board, speaker circuit
Parts:
- added C10: 1uF, SparkFun-Capacitors:CAP0805
- added C101, C102, C8, C9, CBOOT1, CBOOT2, CCLAMP1, CCLAMP2, CCOMM1, CCOMM2: (no value), SparkFun-Capacitors:CAP0805
- added C11, C12: 0.1uF, SparkFun-Capacitors:CAP0805
- added D4: BLUE, SparkFun-LED:LED-BLUE0603
- added FRAME2, FRAME3: FRAME-LETTERNO_PACKAGE, SparkFun-Aesthetics:FRAME-LETTERNO_PACKAGE
- added R4, R5, R6: (no value), SparkFun-Passives:RESISTOR0805-RES
- added R7, R8: 150k, SparkFun-Passives:RESISTOR0805-RES
- added THM2: (no value), BB8:THM
- added U2: TPA2005D1DGN, SparkFun-AnalogIC:TPA2005D1DGN
- added WPC-RX1: BQ51013B-20VQFN, BB8:BQ51013B-20VQFN
Connections:
- new net AC1: C101.2, C102.1, CBOOT1.1, CCLAMP1.1, CCOMM1.1, WPC-RX1.AC1
- new net AC2: C102.2, CBOOT2.1, CCLAMP2.1, CCOMM2.1
- new net AUDIOIN: C11.1
- new net AUDIO_OUT+: U2.OUT+
- new net AUDIO_OUT-: U2.OUT-
- new net BI-STATE: WPC-RX1.EN1
- new net BI-STATE2: WPC-RX1.EN2
- new net BOOT2: CBOOT2.2
- new net N$16: CCOMM2.2
- new net N$17: CCLAMP2.2
- new net N$18: CCLAMP1.2
- new net N$19: CBOOT1.2
- new net N$20: CCOMM1.2
- new net N$21: C101.1
- new net N$22: R4.1, WPC-RX1.ILIM
- new net N$23: R4.2, R5.1, R6.1, WPC-RX1.FOD
- new net N$24: D4.C, WPC-RX1.!CHG
- new net N$25: C9.1, R6.2, WPC-RX1.RECT
- new net N$26: R7.2, U2.IN+
- new net N$28: C11.2, R7.1
- new net N$30: R8.2, U2.IN-
- new net N$32: C12.1, R8.1
- new net OUT: C8.1, D4.A, WPC-RX1.OUT
- new net SPEAKER_SHUTDOWN: U2.SHUTDOWN
- new net TRI-STATE: THM2.1, WPC-RX1.TS/CTRL
- new net VDD_5V: C10.1
- net GND: now also C10.2, C12.2, C8.2, C9.2, R5.2, THM2.2, U2.GND@1, U2.GND@2, WPC-RX1.PGND
Other:
- note added: "Audio Amplifier"
- note added: "MAX745 Charging Circuit"
- note added: "Wireless Charging Receiver"

Commit message: added more info for boards
Parts:
- added FRAME4: FRAME-LETTERNO_PACKAGE, SparkFun-Aesthetics:FRAME-LETTERNO_PACKAGE
- added J1: BATTERY_CONNDEANS, SparkFun-Connectors:BATTERY_CONNDEANS
- added SD1: 5738-SDCARD, BB8:5738-SDCARD
Connections:
- new net CS: SD1.CS
- new net MISO: SD1.MISO
- new net MOSI: SD1.MOSI
- new net N$27: SD1.VCC
- new net SCK: SD1.CLK
- net GND: now also J1.-, SD1.GND@3, SD1.GND@6
- net N$7: now also J1.+
Other:
- note added: "Coil goes here"
- note added: "Depends on what we want"
- note added: "Input from wireless charger"
- note added: "SD Card Connection (SPI)"
- note added: "Temporary, please replace with whatever you need"
Changed lines of the file:
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@@
 <part name="GND19" library="SparkFun-Aesthetics" deviceset="GND" device=""/>
 <part name="U2" library="SparkFun-AnalogIC" deviceset="TPA2005D1" device="DGN"/>
+<part name="J1" library="SparkFun-Connectors" deviceset="BATTERY_CONN" device="DEANS"/>
+<part name="FRAME4" library="SparkFun-Aesthetics" deviceset="FRAME-LETTER" device="NO_PACKAGE"/>
+<part name="SD1" library="BB8" deviceset="5738-SDCARD" device=""/>
+<part name="SUPPLY1" library="SparkFun-Aesthetics" deviceset="VCC" device=""/>
+<part name="GND20" library="SparkFun-Aesthetics" deviceset="GND" device=""/>
 </parts>
 <sheets>
@@
 <text x="-271.78" y="160.02" size="6.35" layer="94">Wireless Charging Receiver</text>
 <text x="-269.24" y="-30.48" size="6.35" layer="94">Audio Amplifier</text>
+<text x="160.02" y="45.72" size="1.778" layer="97">Temporary, please replace with whatever you need</text>
+<text x="-236.22" y="88.9" size="1.778" layer="97" rot="R90">Coil goes here</text>
+<text x="27.94" y="132.08" size="1.778" layer="97">Input from wireless charger</text>
+<text x="93.98" y="40.64" size="1.778" layer="97" rot="R270">Depends on what we want</text>
+<text x="-17.78" y="-30.48" size="6.35" layer="94">SD Card Connection (SPI)</text>
 </plain>
 <instances>
@@
 <instance part="GND19" gate="1" x="-119.38" y="-78.74"/>
 <instance part="U2" gate="G$1" x="-160.02" y="-81.28"/>
+<instance part="J1" gate="G$1" x="177.8" y="55.88"/>
+<instance part="FRAME4" gate="G$1" x="-22.86" y="-203.2"/>
+<instance part="FRAME4" gate="V" x="124.46" y="-203.2"/>
+<instance part="SD1" gate="G$1" x="83.82" y="-101.6"/>
+<instance part="SUPPLY1" gate="G$1" x="58.42" y="-76.2"/>
+<instance part="GND20" gate="1" x="63.5" y="-132.08"/>
 </instances>
 <busses>
@@
 <pinref part="GND4" gate="1" pin="GND"/>
 <wire x1="190.5" y1="48.26" x2="190.5" y2="45.72" width="0.1524" layer="91"/>
+<pinref part="J1" gate="G$1" pin="-"/>
+<wire x1="185.42" y1="53.34" x2="190.5" y2="53.34" width="0.1524" layer="91"/>
+<wire x1="190.5" y1="53.34" x2="190.5" y2="48.26" width="0.1524" layer="91"/>
+<junction x="190.5" y="48.26"/>
 </segment>
 <segment>
@@
 <wire x1="-165.1" y1="-99.06" x2="-165.1" y2="-93.98" width="0.1524" layer="91"/>
 <junction x="-152.4" y="-99.06"/>
+</segment>
+<segment>
+<pinref part="SD1" gate="G$1" pin="GND@3"/>
+<pinref part="GND20" gate="1" pin="GND"/>
+<wire x1="71.12" y1="-121.92" x2="63.5" y2="-121.92" width="0.1524" layer="91"/>
+<wire x1="63.5" y1="-121.92" x2="63.5" y2="-127" width="0.1524" layer="91"/>
+<pinref part="SD1" gate="G$1" pin="GND@6"/>
+<wire x1="63.5" y1="-127" x2="63.5" y2="-129.54" width="0.1524" layer="91"/>
+<wire x1="71.12" y1="-127" x2="63.5" y2="-127" width="0.1524" layer="91"/>
+<junction x="63.5" y="-127"/>
 </segment>
 </net>
@@
 <pinref part="C1" gate="G$1" pin="1"/>
 <wire x1="198.12" y1="60.96" x2="198.12" y2="58.42" width="0.1524" layer="91"/>
+<pinref part="J1" gate="G$1" pin="+"/>
+<wire x1="190.5" y1="60.96" x2="190.5" y2="55.88" width="0.1524" layer="91"/>
+<wire x1="190.5" y1="55.88" x2="185.42" y2="55.88" width="0.1524" layer="91"/>
 </segment>
 </net>
@@
 </segment>
 </net>
+<net name="SCK" class="0">
+<segment>
+<pinref part="SD1" gate="G$1" pin="CLK"/>
+<wire x1="71.12" y1="-91.44" x2="58.42" y2="-91.44" width="0.1524" layer="91"/>
+<label x="58.42" y="-91.44" size="1.778" layer="95"/>
+</segment>
+</net>
+<net name="MISO" class="0">
+<segment>
+<pinref part="SD1" gate="G$1" pin="MISO"/>
+<wire x1="71.12" y1="-106.68" x2="58.42" y2="-106.68" width="0.1524" layer="91"/>
+<label x="58.42" y="-106.68" size="1.778" layer="95"/>
+</segment>
+</net>
+<net name="N$27" class="0">
+<segment>
+<pinref part="SD1" gate="G$1" pin="VCC"/>
+<wire x1="71.12" y1="-81.28" x2="58.42" y2="-81.28" width="0.1524" layer="91"/>
+<wire x1="58.42" y1="-81.28" x2="58.42" y2="-76.2" width="0.1524" layer="91"/>
+<pinref part="SUPPLY1" gate="G$1" pin="VCC"/>
+</segment>
+</net>
+<net name="CS" class="0">
+<segment>
+<pinref part="SD1" gate="G$1" pin="CS"/>
+<wire x1="71.12" y1="-86.36" x2="58.42" y2="-86.36" width="0.1524" layer="91"/>
+<label x="58.42" y="-86.36" size="1.778" layer="95"/>
+</segment>
+</net>
+<net name="MOSI" class="0">
+<segment>
+<pinref part="SD1" gate="G$1" pin="MOSI"/>
+<wire x1="71.12" y1="-101.6" x2="58.42" y2="-101.6" width="0.1524" layer="91"/>
+<label x="58.42" y="-101.6" size="1.778" layer="95"/>
+</segment>
+</net>
