File: ChargingCircuit.sch (EAGLE design)
At the start: 49 parts, among them J1 BATTERY_CONNDEANS, M1 IRF7303, U1 MAX745EACSSOP, U2 TPA2005D1DGN

Commit message: Added BQ40Z60 Charging Circuit
Parts:
- removed FRAME1, FRAME2, FRAME3, FRAME4: FRAME-LETTERNO_PACKAGE, SparkFun-Aesthetics:FRAME-LETTERNO_PACKAGE
- added C13, C17: 22pF, SparkFun-Capacitors:CAP0805
- added C14, C15, C16, C18, C19, C20, C21, C24, C25, C26, C28, C29, C30, C31, C32, C33, C34, C35, C36, C37, C38, C39, C40: 0.1uF, SparkFun-Capacitors:CAP0805
- added C22, C23, C27: 2.2uF, SparkFun-Capacitors:CAP0805
- added D5: MBRA140, SparkFun-DiscreteSemi:MBRA140
- added D6: MBRA140, SparkFun-DiscreteSemi:DIODE-SCHOTTKY-MBRA140
- added D7, D8: 1N4148-0805, BB8:1N4148-0805
- added FRAME6, FRAME7, FRAME8, FRAME9: FRAME-LEDGER, SparkFun-Aesthetics:FRAME-LEDGER
- added J2: (no value), SparkFun-Connectors:M04JST
- added L2: 2.2uH, SparkFun-Passives:INDUCTOR0805
- added Q1, Q2, Q3, Q4, Q5, Q6, Q7: CSD17308Q3, BB8:CSD17308Q3
- added R10, R40, R46, R47: 1k, SparkFun-Resistors:RESISTOR0805-RES
- added R13, R14, R17, R18, R19, R37, R38, R39, R41, R42, R45, R9: 100, SparkFun-Resistors:RESISTOR0805-RES
- added R20: 35.63k, SparkFun-Resistors:RESISTOR0805-RES
- added R21: 332k, SparkFun-Resistors:RESISTOR0805-RES
- added R22: 10m, SparkFun-Resistors:RESISTOR0805-RES
- added R23, R32: 10k, SparkFun-Resistors:RESISTOR0805-RES
- added R24, R25, R30, R33, R35, R44: 5.1k, SparkFun-Resistors:RESISTOR0805-RES
- added R26: 1, SparkFun-Resistors:RESISTOR0805-RES
- added R27: 100k, SparkFun-Resistors:RESISTOR0805-RES
- added R28: 2, SparkFun-Resistors:RESISTOR0805-RES
- added R29, R31, R34: 10M, SparkFun-Resistors:RESISTOR0805-RES
- added R36: 10, SparkFun-Resistors:RESISTOR0805-RES
- added R43: 5m, SparkFun-Resistors:RESISTOR0805-RES
- added RT1: 10k-PTC, BB8:THM
- added RT2, RT3, RT4: (no value), BB8:THM
- added U3: BQ40Z60, BB8:BQ40Z60
- added U4: BQ2947, BB8:BQ2947
- added Z1, Z2, Z3: MM3Z75VC, BB8:MM3Z75VC
- THM1: value (none) -> 10K - NTC
- THM2: value (none) -> 10K-NTC
Connections:
- new net ALERT: R9.2
- new net N$29: R10.1, R13.2, Z1.C
- new net N$31: RT1.1, U3.TS1
- new net N$33: RT2.1, U3.TS2
- new net N$34: RT3.1, U3.TS3
- new net N$35: RT4.1, U3.TS4
- new net N$36: R9.1, U3.ALERT/BTP
- new net N$37: Q1.D1, Q3.G1, R24.1, R29.2
- new net N$38: R13.1, U3.SYSPRES
- new net N$39: R14.1, U3.SMBD
- new net N$40: R14.2, R17.1, Z2.C
- new net N$41: C13.1, R20.2, R21.1, U3.VFB
- new net N$42: R24.2, U3.ACFET
- new net N$43: C18.1, C19.2
- new net N$44: R18.1, U3.SMBC
- new net N$45: R18.2, R19.1, Z3.C
- new net N$46: C15.1, C16.2, L2.2, Q6.S1, R22.2, U3.HSRP
- new net N$47: R26.1, U3.VCC
- new net N$48: D6.A, Q1.G1, R23.1
- new net N$50: C20.2, L2.1, Q2.D1, U3.PH
- new net N$51: C20.1, D5.C, U3.BTST
- new net N$52: C21.1, D5.A, U3.REGN
- new net N$53: C23.2, Q3.D1, Q6.D1, R26.2
- new net N$54: R25.1, U3.AFEFUSE
- new net N$55: C26.1, Q7.G1, R25.2, R35.1, R44.2
- new net N$56: Q6.G1, U3.HIDRV
- new net N$57: D6.C, D7.C
- new net N$58: C22.2, R28.2
- new net N$59: Q2.G1, U3.LODRV
- new net N$60: R30.2, U3.DSG
- new net N$61: Q4.G1, R30.1, R31.2
- new net N$62: R32.2, U3.ACP
- new net N$63: Q4.D1, Q5.D1
- new net N$64: C24.2, C25.1
- new net N$65: C24.1, Q5.S1, R34.1
- new net N$66: Q5.G1, R33.1, R34.2
- new net N$67: R33.2, U3.CHG
- new net N$68: C40.1, U4.CD
- new net N$69: J2.1, R36.1, R37.1, R40.2, R45.2
- new net N$70: D8.C, U3.BAT
- new net N$71: D8.A, R36.2
- new net N$72: C27.1, U3.PBI
- new net N$73: C28.1, R37.2, U3.VC4
- new net N$74: C28.2, C29.1, R38.2, U3.VC3
- new net N$75: C29.2, C30.1, R39.2, U3.VC2
- new net N$76: C31.1, U3.VC1
- new net N$77: C32.1, C33.1, R41.2, U3.SRN
- new net N$78: C33.2, C34.1, R42.2, U3.SRP
- new net N$79: R44.1, U4.OUT
- new net N$80: C36.1, R40.1, U4.V4
- new net N$81: J2.2, R38.1, R46.2
- new net N$82: J2.3, R39.1, R47.1
- new net N$83: C35.1, R45.1, U4.VDD
- new net N$84: C36.2, C37.1, R46.1, U4.V3
- new net N$85: C37.2, C39.2, R47.2, U4.V2
- new net N$86: C38.1, U4.V1
- new net PACK+: C18.2, D7.A, Q1.S1, Q3.S1, R27.1, R28.1, R29.1, R32.1
- new net PACK-: R41.1, R43.2
- new net SMBC: R19.2
- new net SMBD: R17.2
- new net SYSPRES: R10.2
- new net SYSTEMLOAD: C13.2, C14.1, C16.1, C17.2, C25.2, Q4.S1, R21.2, R22.1, R31.1, U3.HSRN
- net AC2: now also WPC-RX1.AC2
- net BOOT2: now also WPC-RX1.BOOT2
- net GND: now also C14.2, C15.2, C17.1, C19.1, C21.2, C22.1, C23.1, C26.2, C27.2, C30.2, C31.2, C32.2, C34.2, C35.2, C38.2, C39.1, C40.2, J2.4, Q2.S1, Q7.S1, R20.1, R23.2, R27.2, R35.2, R42.1, R43.1, RT1.2, RT2.2, RT3.2, RT4.2, U3.PGND, U3.VSS, U4.GNDPAD, U4.VSS, WPC-RX1.AD, Z1.A, Z2.A, Z3.A
- net N$16: now also WPC-RX1.COMM2
- net N$17: now also WPC-RX1.CLAMP2
- net N$18: now also WPC-RX1.CLAMP1
- net N$19: now also WPC-RX1.BOOT1
- net N$20: now also WPC-RX1.COMM1
- net VDD_5V: now also U2.VDD
Other:
- note added: "BQ40Z60 Charging Circuit"
- note added: "FUSE GOES HERE"
- note added: "REPLACE WITH BAS16"
- note removed: "rip in peace"
- moved on the sheet: C1, C10, C101, C102, C11, C12, C2, C3, C4, C5, C6, C7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

Commit message: Preliminary work on BQ40Z60, need to short VC3 and VC4, fix VC1
Parts:
- removed C28: 0.1uF, SparkFun-Capacitors:CAP0805
Connections:
- net N$73: no longer C28.1
- net N$74: no longer C28.2
Changed lines of the file:
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@@
 <part name="R41" library="SparkFun-Resistors" deviceset="RESISTOR" device="0805-RES" value="100"/>
 <part name="R42" library="SparkFun-Resistors" deviceset="RESISTOR" device="0805-RES" value="100"/>
-<part name="C28" library="SparkFun-Capacitors" deviceset="CAP" device="0805" value="0.1uF"/>
 <part name="C29" library="SparkFun-Capacitors" deviceset="CAP" device="0805" value="0.1uF"/>
 <part name="C30" library="SparkFun-Capacitors" deviceset="CAP" device="0805" value="0.1uF"/>
@@
 <instance part="R41" gate="G$1" x="-114.3" y="43.18"/>
 <instance part="R42" gate="G$1" x="-114.3" y="33.02"/>
-<instance part="C28" gate="G$1" x="-93.98" y="78.74"/>
 <instance part="C29" gate="G$1" x="-86.36" y="68.58"/>
 <instance part="C30" gate="G$1" x="-93.98" y="58.42"/>
@@
 <segment>
 <pinref part="U3" gate="G$1" pin="VC4"/>
-<wire x1="-60.96" y1="83.82" x2="-93.98" y2="83.82" width="0.1524" layer="91"/>
+<wire x1="-60.96" y1="83.82" x2="-109.22" y2="83.82" width="0.1524" layer="91"/>
 <pinref part="R37" gate="G$1" pin="2"/>
-<pinref part="C28" gate="G$1" pin="1"/>
-<wire x1="-93.98" y1="83.82" x2="-109.22" y2="83.82" width="0.1524" layer="91"/>
-<junction x="-93.98" y="83.82"/>
 </segment>
 </net>
@@
 <wire x1="-86.36" y1="73.66" x2="-93.98" y2="73.66" width="0.1524" layer="91"/>
 <junction x="-86.36" y="73.66"/>
-<pinref part="C28" gate="G$1" pin="2"/>
 <wire x1="-93.98" y1="73.66" x2="-109.22" y2="73.66" width="0.1524" layer="91"/>
 <wire x1="-93.98" y1="76.2" x2="-93.98" y2="73.66" width="0.1524" layer="91"/>
