File: ChargingCircuit.brd (EAGLE design)
At the start: 100 x 80 mm, 134 parts, among them J1 BATTERY_CONNDEANS, M1 IRF7303, Q1 CSD17308Q3, Q2 CSD17308Q3, Q3 CSD17308Q3, Q4 CSD17308Q3, Q5 CSD17308Q3, Q6 CSD17308Q3, Q7 CSD17308Q3, U1 MAX745EACSSOP, U2 TPA2005D1DGN, U3 BQ40Z60, U4 BQ2947

Commit message: Preliminary work on BQ40Z60, need to short VC3 and VC4, fix VC1
Parts:
- removed C28: 0.1uF, SparkFun-Capacitors:0805
Connections:
- net N$73: no longer C28.1
- net N$74: no longer C28.2
Changed lines of the file:
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@@
 <element name="R41" library="SparkFun-Resistors" package="0805" value="100" x="-332.74" y="-140.97"/>
 <element name="R42" library="SparkFun-Resistors" package="0805" value="100" x="-336.55" y="-140.97"/>
-<element name="C28" library="SparkFun-Capacitors" package="0805" value="0.1uF" x="-340.36" y="-140.97"/>
 <element name="C29" library="SparkFun-Capacitors" package="0805" value="0.1uF" x="-344.17" y="-140.97"/>
 <element name="C30" library="SparkFun-Capacitors" package="0805" value="0.1uF" x="-347.98" y="-140.97"/>
@@
 <contactref element="U3" pad="P$3"/>
 <contactref element="R37" pad="2"/>
-<contactref element="C28" pad="1"/>
-<wire x1="-316.6" y1="-140.97" x2="-341.26" y2="-140.97" width="0" layer="19" extent="1-1"/>
 <wire x1="-122.67" y1="-50.865" x2="-316.6" y2="-140.97" width="0" layer="19" extent="1-1"/>
 </signal>
@@
 <contactref element="R38" pad="2"/>
 <contactref element="C29" pad="1"/>
-<contactref element="C28" pad="2"/>
-<wire x1="-339.46" y1="-140.97" x2="-345.07" y2="-140.97" width="0" layer="19" extent="1-1"/>
-<wire x1="-320.41" y1="-140.97" x2="-339.46" y2="-140.97" width="0" layer="19" extent="1-1"/>
+<wire x1="-320.41" y1="-140.97" x2="-345.07" y2="-140.97" width="0" layer="19" extent="1-1"/>
 <wire x1="-122.17" y1="-50.865" x2="-320.41" y2="-140.97" width="0" layer="19" extent="1-1"/>
 </signal>
